Commit message: Final robot shape

File: robot_arm/urdf/lp.xacro (robot description, xacro)
@@ -3,3 +3,9 @@
     <xacro:property name="l00" value="base_link"/>
     <xacro:property name="l01" value="link_01"/>
+    <xacro:property name="l02" value="link_02"/>
+    <xacro:property name="l03" value="link_03"/>
+    <xacro:property name="l04" value="link_04"/>
+    <xacro:property name="l05" value="link_05"/>
+    <xacro:property name="l06" value="link_06"/>
+    <xacro:property name="l07" value="link_07"/>
 </robot>

File: robot_arm/urdf/rm.xacro (robot description, xacro)
@@ -5,11 +5,53 @@
     <xacro:x_link_box name="${l00}"
     origin_xyz="0 0 0"  origin_rpy="0 0 0"
-    size="1 1 3"/>
+    size="2 2 4"/>
     <xacro:x_joint name="${l00}+${l01}" type="revolute"
-    axis="0 0 1"    limit_low="-3.14"   limit_up="3.14" limit_eff="1000"    limit_vel="0.5"
-    origin_xyz="0 0 0.5"    origin_rpy="0 0 0"
+    axis="0 1 0"    limit_low="-3.14"   limit_up="3.14" limit_eff="1000"    limit_vel="0.5"
+    origin_xyz="0 0 1"    origin_rpy="0 0 0"
     parent="${l00}"  child="${l01}"/>
     <xacro:x_link_box name="${l01}"
-    origin_xyz="0 0 0.2"  origin_rpy="0 0 0"
+    origin_xyz="0 1.5 0"  origin_rpy="0 0 0"
     size="1 1 1"/>
+    <xacro:x_joint name="${l01}+${l02}" type="revolute"
+    axis="1 0 0"    limit_low="-3.14"   limit_up="3.14" limit_eff="1000"    limit_vel="0.5"
+    origin_xyz="0 1.5 -0.5"    origin_rpy="0 0 0"
+    parent="${l01}"  child="${l02}"/>
+    <xacro:x_link_ball name="${l02}"
+    origin_xyz="0 0 0" origin_rpy="0 0 0"
+    radius="0.4"/>
+    <xacro:x_joint name="${l02}+${l03}" type="revolute"
+    axis="0 0 1"    limit_low="0"   limit_up="0" limit_eff="1000"    limit_vel="0.5"
+    origin_xyz="0 0 -0.5"    origin_rpy="0 0 0"
+    parent="${l02}"  child="${l03}"/>
+    <xacro:x_link_cylinder name="${l03}"
+    origin_xyz="0 0 0" origin_rpy="0 0 0"
+    radius="0.3" length="1"/>
+    <xacro:x_joint name="${l03}+${l04}" type="revolute"
+    axis="0 0 1"    limit_low="-3.14"   limit_up="3.14" limit_eff="1000"    limit_vel="0.5"
+    origin_xyz="0 0 -0.5"    origin_rpy="0 0 0"
+    parent="${l03}"  child="${l04}"/>
+    <xacro:x_link_ball name="${l04}"
+    origin_xyz="0 0 0" origin_rpy="0 0 0"
+    radius="0.3"/>
+    <xacro:x_joint name="${l04}+${l05}" type="revolute"
+    axis="0 1 0"    limit_low="-3.14"   limit_up="3.14" limit_eff="1000"    limit_vel="0.5"
+    origin_xyz="0 0 0"    origin_rpy="0 0 0"
+    parent="${l04}"  child="${l05}"/>
+    <xacro:x_link_cylinder name="${l05}"
+    origin_xyz="0 0 -0.4" origin_rpy="0 0 0"
+    radius="0.25" length="0.75"/>
+    <xacro:x_joint name="${l05}+${l06}" type="revolute"
+    axis="1 0 0"    limit_low="-3.14"   limit_up="3.14" limit_eff="1000"    limit_vel="0.5"
+    origin_xyz="0 0 -0.75"    origin_rpy="0 0 0"
+    parent="${l05}"  child="${l06}"/>
+    <xacro:x_link_ball name="${l06}"
+    origin_xyz="0 0 0" origin_rpy="0 0 0"
+    radius="0.25"/>
+    <xacro:x_joint name="${l06}+${l07}" type="revolute"
+    axis="0 1 0"    limit_low="-3.14"   limit_up="3.14" limit_eff="1000"    limit_vel="0.5"
+    origin_xyz="0 0 -0.25"    origin_rpy="0 0 0"
+    parent="${l06}"  child="${l07}"/>
+    <xacro:x_link_box name="${l07}"
+    origin_xyz="0 0 0"  origin_rpy="0 0 0"
+    size="0.3 0.3 0.3"/>
 </robot>

Commit message: Added first parts of fingers

File: robot_arm/urdf/lp.xacro (robot description, xacro)
@@ -9,3 +9,9 @@
     <xacro:property name="l06" value="link_06"/>
     <xacro:property name="l07" value="link_07"/>
+    <xacro:property name="l08" value="link_08"/>
+    <xacro:property name="l09" value="link_09"/>
+    <xacro:property name="l10" value="link_10"/>
+    <xacro:property name="l11" value="link_11"/>
+    <xacro:property name="l12" value="link_12"/>
+    <xacro:property name="l13" value="link_13"/>
 </robot>

File: robot_arm/urdf/rm.xacro (robot description, xacro)
@@ -43,15 +43,39 @@
     <xacro:x_joint name="${l05}+${l06}" type="revolute"
     axis="1 0 0"    limit_low="-3.14"   limit_up="3.14" limit_eff="1000"    limit_vel="0.5"
-    origin_xyz="0 0 -0.75"    origin_rpy="0 0 0"
+    origin_xyz="0 0 -0.80"    origin_rpy="0 0 0"
     parent="${l05}"  child="${l06}"/>
     <xacro:x_link_ball name="${l06}"
     origin_xyz="0 0 0" origin_rpy="0 0 0"
-    radius="0.25"/>
+    radius="0.20"/>
     <xacro:x_joint name="${l06}+${l07}" type="revolute"
-    axis="0 1 0"    limit_low="-3.14"   limit_up="3.14" limit_eff="1000"    limit_vel="0.5"
-    origin_xyz="0 0 0"    origin_rpy="0 0 0"
+    axis="0 0 1"    limit_low="-3.14"   limit_up="3.14" limit_eff="1000"    limit_vel="0.5"
+    origin_xyz="0 0 -0.1"    origin_rpy="0 0 0"
     parent="${l06}"  child="${l07}"/>
     <xacro:x_link_box name="${l07}"
-    origin_xyz="0 0 -0.4"  origin_rpy="0 0 0"
-    size="0.3 0.3 0.5"/>
+    origin_xyz="0 0 -0.1"  origin_rpy="0 0 0"
+    size="0.3 0.2 0.4"/>
+    <!-- FINGER 1 -->
+    <xacro:x_joint name="${l07}+${l08}" type="revolute"
+    axis="1 0 0"    limit_low="-3.14"   limit_up="3.14" limit_eff="1000"    limit_vel="0.5"
+    origin_xyz="0.08 0.08 -0.3"    origin_rpy="0 0 0"
+    parent="${l07}"  child="${l08}"/>
+    <xacro:x_link_box name="${l08}"
+    origin_xyz="0 0 -0.1" origin_rpy="0 0 0"
+    size="0.1 0.05 0.2"/>
+    <!-- FINGER 2 -->
+    <xacro:x_joint name="${l07}+${l09}" type="revolute"
+    axis="1 0 0"    limit_low="-3.14"   limit_up="3.14" limit_eff="1000"    limit_vel="0.5"
+    origin_xyz="0.08 0.08 -0.3"    origin_rpy="0 0 0"
+    parent="${l07}"  child="${l09}"/>
+    <xacro:x_link_box name="${l09}"
+    origin_xyz="-0.17 0 -0.1" origin_rpy="0 0 0"
+    size="0.1 0.05 0.2"/>
+    <!-- FINGER 3 -->
+    <xacro:x_joint name="${l07}+${l10}" type="revolute"
+    axis="1 0 0"    limit_low="-3.14"   limit_up="3.14" limit_eff="1000"    limit_vel="0.5"
+    origin_xyz="0.08 -0.06 -0.3"    origin_rpy="0 0 0"
+    parent="${l07}"  child="${l10}"/>
+    <xacro:x_link_box name="${l10}"
+    origin_xyz="0 0 -0.1" origin_rpy="0 0 0"
+    size="0.1 0.05 0.2"/>
 </robot>

Commit message: Changed names

File: robot_arm/urdf/lp.xacro (robot description, xacro)
@@ -15,3 +15,6 @@
     <xacro:property name="l12" value="link_12"/>
     <xacro:property name="l13" value="link_13"/>
+    <xacro:property name="l14" value="link_14"/>
+    <xacro:property name="l15" value="link_15"/>
+    <xacro:property name="l16" value="link_16"/>
 </robot>

File: robot_arm/urdf/rm.xacro (robot description, xacro)
@@ -6,5 +6,5 @@
     origin_xyz="0 0 0"  origin_rpy="0 0 0"
     size="2 2 4"/>
-    <xacro:x_joint name="${l00}+${l01}" type="revolute"
+    <xacro:x_joint name="Shoulder_Up_Down" type="revolute"
     axis="0 1 0"    limit_low="-3.14"   limit_up="3.14" limit_eff="1000"    limit_vel="0.5"
     origin_xyz="0 0 1"    origin_rpy="0 0 0"
@@ -13,5 +13,5 @@
     origin_xyz="0 1.5 0"  origin_rpy="0 0 0"
     size="1 1 1"/>
-    <xacro:x_joint name="${l01}+${l02}" type="revolute"
+    <xacro:x_joint name="Shoulder_Left_Right" type="revolute"
     axis="1 0 0"    limit_low="-3.14"   limit_up="3.14" limit_eff="1000"    limit_vel="0.5"
     origin_xyz="0 1.5 -0.5"    origin_rpy="0 0 0"
@@ -20,5 +20,5 @@
     origin_xyz="0 0 0" origin_rpy="0 0 0"
     radius="0.4"/>
-    <xacro:x_joint name="${l02}+${l03}" type="revolute"
+    <xacro:x_joint name="Shoulder_Rotate_1" type="revolute"
     axis="0 0 1"    limit_low="0"   limit_up="0" limit_eff="1000"    limit_vel="0.5"
     origin_xyz="0 0 -0.5"    origin_rpy="0 0 0"
@@ -27,5 +27,5 @@
     origin_xyz="0 0 0" origin_rpy="0 0 0"
     radius="0.3" length="1"/>
-    <xacro:x_joint name="${l03}+${l04}" type="revolute"
+    <xacro:x_joint name="Shoulder_Rotate" type="revolute"
     axis="0 0 1"    limit_low="-3.14"   limit_up="3.14" limit_eff="1000"    limit_vel="0.5"
     origin_xyz="0 0 -0.5"    origin_rpy="0 0 0"
@@ -34,5 +34,5 @@
     origin_xyz="0 0 0" origin_rpy="0 0 0"
     radius="0.3"/>
-    <xacro:x_joint name="${l04}+${l05}" type="revolute"
+    <xacro:x_joint name="Elbow_Up_Down" type="revolute"
     axis="0 1 0"    limit_low="-3.14"   limit_up="3.14" limit_eff="1000"    limit_vel="0.5"
     origin_xyz="0 0 0"    origin_rpy="0 0 0"
@@ -41,5 +41,5 @@
     origin_xyz="0 0 -0.4" origin_rpy="0 0 0"
     radius="0.25" length="0.75"/>
-    <xacro:x_joint name="${l05}+${l06}" type="revolute"
+    <xacro:x_joint name="Wrist_Left_Right" type="revolute"
     axis="1 0 0"    limit_low="-3.14"   limit_up="3.14" limit_eff="1000"    limit_vel="0.5"
     origin_xyz="0 0 -0.80"    origin_rpy="0 0 0"
@@ -48,5 +48,5 @@
     origin_xyz="0 0 0" origin_rpy="0 0 0"
     radius="0.20"/>
-    <xacro:x_joint name="${l06}+${l07}" type="revolute"
+    <xacro:x_joint name="Wrist_Rotate" type="revolute"
     axis="0 0 1"    limit_low="-3.14"   limit_up="3.14" limit_eff="1000"    limit_vel="0.5"
     origin_xyz="0 0 -0.1"    origin_rpy="0 0 0"
@@ -55,6 +55,6 @@
     origin_xyz="0 0 -0.1"  origin_rpy="0 0 0"
     size="0.3 0.2 0.4"/>
-    <!-- FINGER 1 -->
-    <xacro:x_joint name="${l07}+${l08}" type="revolute"
+    <!-- FINGER 1 A -->
+    <xacro:x_joint name="Index_1" type="revolute"
     axis="1 0 0"    limit_low="-3.14"   limit_up="3.14" limit_eff="1000"    limit_vel="0.5"
     origin_xyz="0.08 0.08 -0.3"    origin_rpy="0 0 0"
@@ -63,6 +63,17 @@
     origin_xyz="0 0 -0.1" origin_rpy="0 0 0"
     size="0.1 0.05 0.2"/>
-    <!-- FINGER 2 -->
-    <xacro:x_joint name="${l07}+${l09}" type="revolute"
+    <!-- FINGER 1 B -->
+    <!-- <xacro:x_joint name="${l07}+${l14}" type="revolute"
+    axis="1 0 0"    limit_low="-3.14"   limit_up="3.14" limit_eff="1000"    limit_vel="0.5"
+    origin_xyz="0.08 0.08 -0.5"    origin_rpy="0 0 0"
+    parent="${l07}"  child="${l14}"/>
+    <xacro:x_link_ball name="${l14}"
+    origin_xyz="0 0 0" origin_rpy="0 0 0"
+    radius="0.05"/> -->
+    <!-- <xacro:x_link_box name="${l11}"
+    origin_xyz="0 0 -0.1" origin_rpy="0 0 0"
+    size="0.1 0.05 0.2"/> -->
+    <!-- FINGER 2 A -->
+    <xacro:x_joint name="Ring_1" type="revolute"
     axis="1 0 0"    limit_low="-3.14"   limit_up="3.14" limit_eff="1000"    limit_vel="0.5"
     origin_xyz="0.08 0.08 -0.3"    origin_rpy="0 0 0"
@@ -71,11 +82,33 @@
     origin_xyz="-0.17 0 -0.1" origin_rpy="0 0 0"
     size="0.1 0.05 0.2"/>
-    <!-- FINGER 3 -->
-    <xacro:x_joint name="${l07}+${l10}" type="revolute"
+    <!-- FINGER 2 B -->
+    <!-- <xacro:x_joint name="${l07}+${l15}" type="revolute"
+    axis="1 0 0"    limit_low="-3.14"   limit_up="3.14" limit_eff="1000"    limit_vel="0.5"
+    origin_xyz="0.08 0.08 -0.5"    origin_rpy="0 0 0"
+    parent="${l07}"  child="${l15}"/>
+    <xacro:x_link_ball name="${l15}"
+    origin_xyz="-0.17 0 0" origin_rpy="0 0 0"
+    radius="0.05"/> -->
+    <!-- <xacro:x_link_box name="${l12}"
+    origin_xyz="-0.17 0 -0.1" origin_rpy="0 0 0"
+    size="0.1 0.05 0.2"/> -->
+    <!-- FINGER 3 A-->
+    <xacro:x_joint name="Thumb_1" type="revolute"
     axis="1 0 0"    limit_low="-3.14"   limit_up="3.14" limit_eff="1000"    limit_vel="0.5"
     origin_xyz="0.08 -0.06 -0.3"    origin_rpy="0 0 0"
     parent="${l07}"  child="${l10}"/>
     <xacro:x_link_box name="${l10}"
-    origin_xyz="0 0 -0.1" origin_rpy="0 0 0"
+    origin_xyz="-0.05 0 -0.1" origin_rpy="0 0 0"
     size="0.1 0.05 0.2"/>
+    <!-- FINGER 3 B-->
+    <!-- <xacro:x_joint name="${l07}+${l16}" type="revolute"
+    axis="1 0 0"    limit_low="-3.14"   limit_up="3.14" limit_eff="1000"    limit_vel="0.5"
+    origin_xyz="0.08 -0.06 -0.5"    origin_rpy="0 0 0"
+    parent="${l07}"  child="${l16}"/>
+    <xacro:x_link_ball name="${l16}"
+    origin_xyz="0 0 0" origin_rpy="0 0 0"
+    radius="0.05"/> -->
+    <!-- <xacro:x_link_box name="${l13}"
+    origin_xyz="-0.05 0 -0.1" origin_rpy="0 0 0"
+    size="0.1 0.05 0.2"/> -->
 </robot>
