Commit message: README update

File: robot_arm/urdf/rm.xacro (robot description, xacro)
@@ -1,26 +1,15 @@
 <?xml version="1.0"?>
 <robot name="rm" xmlns:xacro="http://www.ros.org/wiki/xacro">
-    <link name="base_link">
-        <visual>
-            <origin xyz="0.0 0.0 0.0" rpy="0.0 0.0 0.0"/>
-            <geometry>
-                <box size="1 1 1"/>
-            </geometry>
-        </visual>
-    </link>
-    <joint name="base_link__link_01" type="revolute">
-        <axis xyz="0 0 1"/>
-        <limit lower="-3.14" upper="3.14" effort="1000.0" velocity="0.5"/>
-        <origin xyz="0.0 0.0 0.5" rpy="0.0 0.0 0.0"/>
-        <parent link="base_link"/>
-        <child link="link_01"/>
-    </joint>
-    <link name="link_01">
-        <visual>
-            <origin xyz="0.0 0.0 0.2" rpy="0.0 0.0 0.0"/>
-            <geometry>
-                <cylinder radius="0.35" length="0.4"/>
-            </geometry>
-        </visual>
-    </link>
+    <xacro:include filename="$(find robot_arm)/urdf/jl.xacro"/>
+    <xacro:include filename="$(find robot_arm)/urdf/lp.xacro"/>
+    <xacro:x_link_box name="${l00}"
+    origin_xyz="0 0 0"  origin_rpy="0 0 0"
+    size="1 1 3"/>
+    <xacro:x_joint name="${l00}+${l01}" type="revolute"
+    axis="0 0 1"    limit_low="-3.14"   limit_up="3.14" limit_eff="1000"    limit_vel="0.5"
+    origin_xyz="0 0 0.5"    origin_rpy="0 0 0"
+    parent="${l00}"  child="${l01}"/>
+    <xacro:x_link_box name="${l01}"
+    origin_xyz="0 0 0.2"  origin_rpy="0 0 0"
+    size="1 1 1"/>
 </robot>

Commit message: Addedx inertia, mass and movement. Need to be reevaluated

File: robot_arm/urdf/rm.xacro (robot description, xacro)
@@ -3,13 +3,28 @@
     <xacro:include filename="$(find robot_arm)/urdf/jl.xacro"/>
     <xacro:include filename="$(find robot_arm)/urdf/lp.xacro"/>
+    <!-- Opis robota -->
     <xacro:x_link_box name="${l00}"
     origin_xyz="0 0 0"  origin_rpy="0 0 0"
+    mass = "4096"
+    ixx="1" ixy="0" ixz="0" iyy="1" izz="2" iyz="0"
     size="2 2 4"/>
     <xacro:x_joint name="Shoulder_Up_Down" type="revolute"
-    axis="0 1 0"    limit_low="-3.14"   limit_up="3.14" limit_eff="1000"    limit_vel="0.5"
+    axis="0 1 0"    limit_low="-3.14"   limit_up="3.14" limit_eff="1000"    limit_vel="0.2"
     origin_xyz="0 0 1"    origin_rpy="0 0 0"
     parent="${l00}"  child="${l01}"/>
+    <transmission name="trans_Shoulder_Up_Down">
+        <type>transmission_interface/SimpleTransmission</type>
+        <joint name="Shoulder_Up_Down">
+            <hardwareInterface>hardware_interface/EffortJointInterface</hardwareInterface>
+        </joint>
+        <actuator name="motor_Shoulder_Up_Down">
+            <hardwareInterface>hardware_interface/EffortJointInterface</hardwareInterface>
+            <mechanicalReduction>1</mechanicalReduction>
+        </actuator>
+    </transmission>
     <xacro:x_link_box name="${l01}"
     origin_xyz="0 1.5 0"  origin_rpy="0 0 0"
+    mass = "128"
+    ixx="0.5" ixy="0" ixz="0" iyy="0.5" izz="0.5" iyz="0"
     size="1 1 1"/>
     <xacro:x_joint name="Shoulder_Left_Right" type="revolute"
@@ -19,4 +34,6 @@
     <xacro:x_link_ball name="${l02}"
     origin_xyz="0 0 0" origin_rpy="0 0 0"
+    mass = "64"
+    ixx="0.2" ixy="0" ixz="0" iyy="0.2" izz="0.2" iyz="0"
     radius="0.4"/>
     <xacro:x_joint name="Shoulder_Rotate_1" type="revolute"
@@ -26,4 +43,6 @@
     <xacro:x_link_cylinder name="${l03}"
     origin_xyz="0 0 0" origin_rpy="0 0 0"
+    mass = "64"
+    ixx="0.15" ixy="0" ixz="0" iyy="0.15" izz="0.5" iyz="0"
     radius="0.3" length="1"/>
     <xacro:x_joint name="Shoulder_Rotate" type="revolute"
@@ -33,4 +52,6 @@
     <xacro:x_link_ball name="${l04}"
     origin_xyz="0 0 0" origin_rpy="0 0 0"
+    mass = "16"
+    ixx="0.15" ixy="0" ixz="0" iyy="0.15" izz="0.15" iyz="0"
     radius="0.3"/>
     <xacro:x_joint name="Elbow_Up_Down" type="revolute"
@@ -40,4 +61,6 @@
     <xacro:x_link_cylinder name="${l05}"
     origin_xyz="0 0 -0.4" origin_rpy="0 0 0"
+    mass = "32"
+    ixx="0.125" ixy="0" ixz="0" iyy="0.125" izz="0.375" iyz="0"
     radius="0.25" length="0.75"/>
     <xacro:x_joint name="Wrist_Left_Right" type="revolute"
@@ -47,4 +70,6 @@
     <xacro:x_link_ball name="${l06}"
     origin_xyz="0 0 0" origin_rpy="0 0 0"
+    mass = "16"
+    ixx="0.125" ixy="0" ixz="0" iyy="0.125" izz="0.375" iyz="0"
     radius="0.20"/>
     <xacro:x_joint name="Wrist_Rotate" type="revolute"
@@ -54,4 +79,6 @@
     <xacro:x_link_box name="${l07}"
     origin_xyz="0 0 -0.1"  origin_rpy="0 0 0"
+    mass = "16"
+    ixx="0.15" ixy="0" ixz="0" iyy="0.1" izz="0.2" iyz="0"
     size="0.3 0.2 0.4"/>
     <!-- FINGER 1 A -->
@@ -62,4 +89,6 @@
     <xacro:x_link_box name="${l08}"
     origin_xyz="0 0 -0.1" origin_rpy="0 0 0"
+    mass = "4"
+    ixx="0.05" ixy="0" ixz="0" iyy="0.025" izz="0.1" iyz="0"
     size="0.1 0.05 0.2"/>
     <!-- FINGER 1 B -->
@@ -68,9 +97,8 @@
     origin_xyz="0 0 -0.2"    origin_rpy="0 0 0"
     parent="${l08}"  child="${l11}"/>
-    <!-- <xacro:x_link_ball name="${l14}"
-    origin_xyz="0 0 0" origin_rpy="0 0 0"
-    radius="0.05"/>  -->
     <xacro:x_link_box name="${l11}"
     origin_xyz="0 0 -0.1" origin_rpy="0 0 0"
+    mass = "2"
+    ixx="0.05" ixy="0" ixz="0" iyy="0.025" izz="0.1" iyz="0"
     size="0.1 0.05 0.2"/>
     <!-- FINGER 2 A -->
@@ -81,4 +109,6 @@
     <xacro:x_link_box name="${l09}"
     origin_xyz="-0.17 0 -0.1" origin_rpy="0 0 0"
+    mass = "4"
+    ixx="0.05" ixy="0" ixz="0" iyy="0.025" izz="0.1" iyz="0"
     size="0.1 0.05 0.2"/>
     <!-- FINGER 2 B -->
@@ -87,9 +117,8 @@
     origin_xyz="-0.17 0 -0.2"    origin_rpy="0 0 0"
     parent="${l09}"  child="${l12}"/>
-    <!-- <xacro:x_link_ball name="${l15}"
-    origin_xyz="-0.17 0 0" origin_rpy="0 0 0"
-    radius="0.05"/>  -->
     <xacro:x_link_box name="${l12}"
     origin_xyz="0 0 -0.1" origin_rpy="0 0 0"
+    mass = "2"
+    ixx="0.05" ixy="0" ixz="0" iyy="0.025" izz="0.1" iyz="0"
     size="0.1 0.05 0.2"/>
     <!-- FINGER 3 A-->
@@ -100,4 +129,6 @@
     <xacro:x_link_box name="${l10}"
     origin_xyz="-0.05 0 -0.1" origin_rpy="0 0 0"
+    mass = "4"
+    ixx="0.05" ixy="0" ixz="0" iyy="0.025" izz="0.1" iyz="0"
     size="0.1 0.05 0.2"/>
     <!-- FINGER 3 B-->
@@ -106,9 +137,12 @@
     origin_xyz="0 0 -0.2"    origin_rpy="0 0 0"
     parent="${l10}"  child="${l13}"/>
-    <!-- <xacro:x_link_ball name="${l16}"
-    origin_xyz="0 0 0" origin_rpy="0 0 0"
-    radius="0.05"/> -->
     <xacro:x_link_box name="${l13}"
     origin_xyz="-0.05 0 -0.1" origin_rpy="0 0 0"
+    mass = "2"
+    ixx="0.05" ixy="0" ixz="0" iyy="0.025" izz="0.1" iyz="0"
     size="0.1 0.05 0.2"/>
+    <gazebo>
+        <plugin name="gazebo_ros_control" filename="libgazebo_ros_control.so">
+        </plugin>
+    </gazebo>
 </robot>

Commit message: Error with controller

File: robot_arm/urdf/rm.xacro (robot description, xacro)
@@ -9,14 +9,14 @@
     ixx="1" ixy="0" ixz="0" iyy="1" izz="2" iyz="0"
     size="2 2 4"/>
-    <xacro:x_joint name="Shoulder_Up_Down" type="revolute"
+    <xacro:x_joint name="base_link__link_01" type="revolute"
     axis="0 1 0"    limit_low="-3.14"   limit_up="3.14" limit_eff="1000"    limit_vel="0.2"
     origin_xyz="0 0 1"    origin_rpy="0 0 0"
     parent="${l00}"  child="${l01}"/>
-    <transmission name="trans_Shoulder_Up_Down">
+    <transmission name="trans_base_link__link_01">
         <type>transmission_interface/SimpleTransmission</type>
-        <joint name="Shoulder_Up_Down">
+        <joint name="base_link__link_01">
             <hardwareInterface>hardware_interface/EffortJointInterface</hardwareInterface>
         </joint>
-        <actuator name="motor_Shoulder_Up_Down">
+        <actuator name="motor_base_link__link_01">
             <hardwareInterface>hardware_interface/EffortJointInterface</hardwareInterface>
             <mechanicalReduction>1</mechanicalReduction>
@@ -28,5 +28,5 @@
     ixx="0.5" ixy="0" ixz="0" iyy="0.5" izz="0.5" iyz="0"
     size="1 1 1"/>
-    <xacro:x_joint name="Shoulder_Left_Right" type="revolute"
+<!--     <xacro:x_joint name="Shoulder_Left_Right" type="revolute"
     axis="1 0 0"    limit_low="-3.14"   limit_up="3.14" limit_eff="1000"    limit_vel="0.5"
     origin_xyz="0 1.5 -0.5"    origin_rpy="0 0 0"
@@ -82,5 +82,5 @@
     ixx="0.15" ixy="0" ixz="0" iyy="0.1" izz="0.2" iyz="0"
     size="0.3 0.2 0.4"/>
-    <!-- FINGER 1 A -->
+     FINGER 1 A
     <xacro:x_joint name="Index_1" type="revolute"
     axis="1 0 0"    limit_low="-3.14"   limit_up="3.14" limit_eff="1000"    limit_vel="0.5"
@@ -92,6 +92,6 @@
     ixx="0.05" ixy="0" ixz="0" iyy="0.025" izz="0.1" iyz="0"
     size="0.1 0.05 0.2"/>
-    <!-- FINGER 1 B -->
-     <xacro:x_joint name="Index_2" type="revolute"
+     FINGER 1 B
+    <xacro:x_joint name="Index_2" type="revolute"
     axis="1 0 0"    limit_low="-3.14"   limit_up="3.14" limit_eff="1000"    limit_vel="0.5"
     origin_xyz="0 0 -0.2"    origin_rpy="0 0 0"
@@ -102,5 +102,5 @@
     ixx="0.05" ixy="0" ixz="0" iyy="0.025" izz="0.1" iyz="0"
     size="0.1 0.05 0.2"/>
-    <!-- FINGER 2 A -->
+     FINGER 2 A
     <xacro:x_joint name="Ring_1" type="revolute"
     axis="1 0 0"    limit_low="-3.14"   limit_up="3.14" limit_eff="1000"    limit_vel="0.5"
@@ -112,5 +112,5 @@
     ixx="0.05" ixy="0" ixz="0" iyy="0.025" izz="0.1" iyz="0"
     size="0.1 0.05 0.2"/>
-    <!-- FINGER 2 B -->
+     FINGER 2 B
     <xacro:x_joint name="Ring_2" type="revolute"
     axis="1 0 0"    limit_low="-3.14"   limit_up="3.14" limit_eff="1000"    limit_vel="0.5"
@@ -122,5 +122,5 @@
     ixx="0.05" ixy="0" ixz="0" iyy="0.025" izz="0.1" iyz="0"
     size="0.1 0.05 0.2"/>
-    <!-- FINGER 3 A-->
+     FINGER 3 A
     <xacro:x_joint name="Thumb_1" type="revolute"
     axis="1 0 0"    limit_low="-3.14"   limit_up="3.14" limit_eff="1000"    limit_vel="0.5"
@@ -132,5 +132,5 @@
     ixx="0.05" ixy="0" ixz="0" iyy="0.025" izz="0.1" iyz="0"
     size="0.1 0.05 0.2"/>
-    <!-- FINGER 3 B-->
+     FINGER 3 B
     <xacro:x_joint name="Thumb_2" type="revolute"
     axis="1 0 0"    limit_low="-3.14"   limit_up="3.14" limit_eff="1000"    limit_vel="0.5"
@@ -141,5 +141,5 @@
     mass = "2"
     ixx="0.05" ixy="0" ixz="0" iyy="0.025" izz="0.1" iyz="0"
-    size="0.1 0.05 0.2"/>
+    size="0.1 0.05 0.2"/> -->
     <gazebo>
         <plugin name="gazebo_ros_control" filename="libgazebo_ros_control.so">
