Commit message: added MoveIt package

File: robot_arm/urdf/backup_rm.xacro (robot description, xacro)
@@ -9,5 +9,5 @@
     origin_xyz="0 0 0"  origin_rpy="0 0 0"
     mass = "4800" size="2 2 6"
-    ixx="16000" ixy="0" ixz="0" iyy="16000" izz="3200" iyz="0"
+    ixx="16000" iyy="16000" izz="3200" iyz="0" ixy="0" ixz="0"
     material="Rust"
     />
@@ -15,5 +15,5 @@
 <!--================================================================================-->
     <xacro:x_joint name="Shoulder_01" type="revolute"
-    axis="0 1 0"    limit_low="-2.97"   limit_up="0.87" limit_eff="10000"  limit_vel="0.5"
+    axis="0 1 0"    limit_low="-2.97"   limit_up="0.87" limit_eff="20000"  limit_vel="1"
     origin_xyz="0 0 2"    origin_rpy="0 0 0"
     parent="${l00}"  child="${l01}"/>
@@ -31,10 +31,10 @@
     origin_xyz="0 1.5 0"  origin_rpy="0 0 0"
     mass = "192" size="1 1 1"
-    ixx="32" ixy="0" ixz="0" iyy="32" izz="32" iyz="0"
+    ixx="16" iyy="16" izz="16" iyz="0" ixy="0" ixz="0"
     material="Rust" />
     <!-- Barka, od siebie do siebie -->
 <!--================================================================================-->
     <xacro:x_joint name="Shoulder_02" type="revolute"
-    axis="1 0 0"    limit_low="-0.35"   limit_up="1.6" limit_eff="10000"    limit_vel="0.5"
+    axis="1 0 0"    limit_low="-0.35"   limit_up="1.6" limit_eff="20000"    limit_vel="1"
     origin_xyz="0 1.5 -0.5"    origin_rpy="0 0 0"
     parent="${l01}"  child="${l02}"/>
@@ -52,5 +52,5 @@
     origin_xyz="0 0 0" origin_rpy="0 0 0"
     mass = "40" radius="0.4"
-    ixx="2.56" ixy="0" ixz="0" iyy="2.56" izz="2.56" iyz="0"
+    ixx="1.28" iyy="1.28" izz="1.28" iyz="0"  ixy="0" ixz="0"
     material="Rust" />
     <!-- Ramię, martwy joint -->
@@ -73,5 +73,5 @@
     origin_xyz="0 0 0" origin_rpy="0 0 0"
     mass = "48" radius="0.3" length="1"
-    ixx="5.08" ixy="0" ixz="0" iyy="5.08" izz="2.16" iyz="0"
+    ixx="17.7" iyy="17.7" izz="1.08" iyz="0"  ixy="0" ixz="0"
     material="Rust" />
     <!-- Łokieć, rotacja -->
@@ -94,10 +94,10 @@
     origin_xyz="0 0 0" origin_rpy="0 0 0"
     mass = "15" radius="0.3"
-    ixx="0.54" ixy="0" ixz="0" iyy="0.54" izz="0.54" iyz="0"
+    ixx="0.54" iyy="0.54" izz="0.54" iyz="0" ixy="0" ixz="0"
     material="Rust" />
     <!-- Łokieć, zgięcie-->
 <!--================================================================================-->
     <xacro:x_joint name="Arm_03" type="revolute"
-    axis="0 1 0"    limit_low="-2.62"   limit_up="0" limit_eff="10000"    limit_vel="0.5"
+    axis="0 1 0"    limit_low="-2.62"   limit_up="0" limit_eff="20000"    limit_vel="1"
     origin_xyz="0 0 0"    origin_rpy="0 0 0"
     parent="${l04}"  child="${l05}"/>
@@ -115,5 +115,5 @@
     origin_xyz="0 0 -0.4" origin_rpy="0 0 0"
     mass = "48" radius="0.25" length="0.75"
-    ixx="9.75" ixy="0" ixz="0" iyy="9.75" izz="1.5" iyz="0"
+    ixx="10" iyy="10" izz="1.5" iyz="0" ixy="0" ixz="0"
     material="Rust" />
     <!-- Nadgarstek, góra dół -->
@@ -136,5 +136,5 @@
     origin_xyz="0 0 0" origin_rpy="0 0 0"
     mass = "15" radius="0.20"
-    ixx="0.24" ixy="0" ixz="0" iyy="0.24" izz="0.24" iyz="0"
+    ixx="0.24" iyy="0.24" izz="0.24" iyz="0" ixy="0" ixz="0"
     material="Rust" />
     <!-- Nadgarstek, rotacyjny -->
@@ -157,5 +157,5 @@
     origin_xyz="0 0 -0.1"  origin_rpy="0 0 0"
     mass = "24" size="0.3 0.2 0.4"
-    ixx="0.5" ixy="0" ixz="0" iyy="0.26" izz="1.36" iyz="0"
+    ixx="0.5" iyy="0.26" izz="4.24" iyz="0"  ixy="0" ixz="0"
     material="Rust" />
      <!-- Palec wskazujący A -->
@@ -178,5 +178,5 @@
     origin_xyz="0 0 -0.1" origin_rpy="0 0 0"
     mass = "4" size="0.1 0.05 0.2"
-    ixx="1" ixy="0" ixz="0" iyy="1" izz="1" iyz="0"
+    ixx="1.344" iyy="0.014" izz="0.02" iyz="0" ixy="0" ixz="0"
     material="Rust" />
     <!-- Palec wskazujący B -->
@@ -199,5 +199,5 @@
     origin_xyz="0 0 -0.1" origin_rpy="0 0 0"
     mass = "4" size="0.1 0.05 0.2"
-    ixx="1" ixy="0" ixz="0" iyy="1" izz="1" iyz="0"
+    ixx="1.344" iyy="0.014" izz="0.02" iyz="0" ixy="0" ixz="0"
     material="Rust" />
    <!--  Palec serdeczny A -->
@@ -220,5 +220,5 @@
     origin_xyz="-0.17 0 -0.1" origin_rpy="0 0 0"
     mass = "4"  size="0.1 0.05 0.2"
-    ixx="1" ixy="0" ixz="0" iyy="1" izz="1" iyz="0"
+    ixx="1.344" iyy="0.014" izz="0.02" iyz="0" ixy="0" ixz="0"
     material="Rust" />
      <!-- Palec serdeczny B -->
@@ -241,5 +241,5 @@
     origin_xyz="0 0 -0.1" origin_rpy="0 0 0"
     mass = "4" size="0.1 0.05 0.2"
-    ixx="1" ixy="0" ixz="0" iyy="1" izz="1" iyz="0"
+    ixx="1.344" iyy="0.014" izz="0.02" iyz="0" ixy="0" ixz="0"
     material="Rust" />
     <!--  Palec kciuk A -->
@@ -262,5 +262,5 @@
     origin_xyz="-0.05 0 -0.1" origin_rpy="0 0 0"
     mass = "4"  size="0.1 0.05 0.2"
-    ixx="1" ixy="0" ixz="0" iyy="1" izz="1" iyz="0"
+    ixx="1.344" iyy="0.014" izz="0.02" iyz="0" ixy="0" ixz="0"
     material="Rust" />
      <!-- Palec kciuk B -->
@@ -283,5 +283,5 @@
     origin_xyz="-0.05 0 -0.1" origin_rpy="0 0 0"
     mass = "4" size="0.1 0.05 0.2"
-    ixx="1" ixy="0" ixz="0" iyy="1" izz="1" iyz="0"
+    ixx="1.344" iyy="0.014" izz="0.02" iyz="0" ixy="0" ixz="0"
     material="Rust" />
     <!-- Plugin -->

File: robot_arm/urdf/jl.xacro (robot description, xacro)
@@ -72,5 +72,5 @@
                 <origin xyz="${origin_xyz}" rpy="${origin_rpy}"/>
                 <geometry>
-                    <sphere radius="${radius}"/>
+                    <sphere radius="0.1"/>
                 </geometry>
             </collision>

File: robot_arm/urdf/rm.xacro (robot description, xacro)
@@ -7,5 +7,5 @@
 <!--================================================================================-->
     <xacro:x_link_box name="${l00}"
-    origin_xyz="0 0 0"  origin_rpy="0 0 0"
+    origin_xyz="0 0 1"  origin_rpy="0 0 0"
     mass = "4800" size="2 2 6"
     ixx="16000" iyy="16000" izz="3200" iyz="0" ixy="0" ixz="0"
@@ -15,6 +15,6 @@
 <!--================================================================================-->
     <xacro:x_joint name="Shoulder_01" type="revolute"
-    axis="0 1 0"    limit_low="-2.97"   limit_up="0.87" limit_eff="20000"  limit_vel="1"
-    origin_xyz="0 0 2"    origin_rpy="0 0 0"
+    axis="0 1 0"    limit_low="-2.97"   limit_up="0.87" limit_eff="30000"  limit_vel="1"
+    origin_xyz="0 0 3"    origin_rpy="0 0 0"
     parent="${l00}"  child="${l01}"/>
     <transmission name="trans_Shoulder_01">
@@ -30,5 +30,5 @@
     <xacro:x_link_box name="${l01}"
     origin_xyz="0 1.5 0"  origin_rpy="0 0 0"
-    mass = "192" size="1 1 1"
+    mass = "192" size="1 0.98 1"
     ixx="16" iyy="16" izz="16" iyz="0" ixy="0" ixz="0"
     material="Rust" />
@@ -36,6 +36,6 @@
 <!--================================================================================-->
     <xacro:x_joint name="Shoulder_02" type="revolute"
-    axis="1 0 0"    limit_low="-0.35"   limit_up="1.6" limit_eff="20000"    limit_vel="1"
-    origin_xyz="0 1.5 -0.5"    origin_rpy="0 0 0"
+    axis="1 0 0"    limit_low="-0.35"   limit_up="1.6" limit_eff="30000"    limit_vel="1"
+    origin_xyz="0 2 -0.5"    origin_rpy="0 0 0"
     parent="${l01}"  child="${l02}"/>
     <transmission name="trans_Shoulder_02">
@@ -58,5 +58,5 @@
     <xacro:x_joint name="Arm_01" type="revolute"
     axis="0 0 1"    limit_low="0"   limit_up="0" limit_eff="10000"    limit_vel="0.5"
-    origin_xyz="0 0 -0.5"    origin_rpy="0 0 0"
+    origin_xyz="0 0 -0.55"    origin_rpy="0 0 0"
     parent="${l02}"  child="${l03}"/>
     <transmission name="trans_Arm_01">
@@ -72,5 +72,5 @@
     <xacro:x_link_cylinder name="${l03}"
     origin_xyz="0 0 0" origin_rpy="0 0 0"
-    mass = "48" radius="0.3" length="1"
+    mass = "48" radius="0.25" length="1"
     ixx="17.7" iyy="17.7" izz="1.08" iyz="0"  ixy="0" ixz="0"
     material="Rust" />
@@ -79,5 +79,5 @@
     <xacro:x_joint name="Arm_02" type="revolute"
     axis="0 0 1"    limit_low="-1.6"   limit_up="1.60" limit_eff="10000"    limit_vel="0.5"
-    origin_xyz="0 0 -0.5"    origin_rpy="0 0 0"
+    origin_xyz="0 0 -0.7"    origin_rpy="0 0 0"
     parent="${l03}"  child="${l04}"/>
     <transmission name="trans_Arm_02">
@@ -113,6 +113,6 @@
     </transmission>
     <xacro:x_link_cylinder name="${l05}"
-    origin_xyz="0 0 -0.4" origin_rpy="0 0 0"
-    mass = "48" radius="0.25" length="0.75"
+    origin_xyz="0 0 -0.6" origin_rpy="0 0 0"
+    mass = "48" radius="0.2" length="0.75"
     ixx="10" iyy="10" izz="1.5" iyz="0" ixy="0" ixz="0"
     material="Rust" />
@@ -121,5 +121,5 @@
     <xacro:x_joint name="Wrist" type="revolute"
     axis="1 0 0"    limit_low="-1.05"   limit_up="0.87" limit_eff="10000"    limit_vel="0.5"
-    origin_xyz="0 0 -0.80"    origin_rpy="0 0 0"
+    origin_xyz="0 0 -1"    origin_rpy="0 0 0"
     parent="${l05}"  child="${l06}"/>
     <transmission name="trans_Wrist">
@@ -134,5 +134,5 @@
     </transmission>
     <xacro:x_link_ball name="${l06}"
-    origin_xyz="0 0 0" origin_rpy="0 0 0"
+    origin_xyz="0 0 -0.05" origin_rpy="0 0 0"
     mass = "15" radius="0.20"
     ixx="0.24" iyy="0.24" izz="0.24" iyz="0" ixy="0" ixz="0"
@@ -155,5 +155,5 @@
     </transmission>
     <xacro:x_link_box name="${l07}"
-    origin_xyz="0 0 -0.1"  origin_rpy="0 0 0"
+    origin_xyz="0 0 -0.25"  origin_rpy="0 0 0"
     mass = "24" size="0.3 0.2 0.4"
     ixx="0.5" iyy="0.26" izz="4.24" iyz="0"  ixy="0" ixz="0"
