Commit message: Added joint andx links inertia and collision scheme

File: robot_arm/urdf/jl.xacro (robot description, xacro)
@@ -10,6 +10,17 @@
         </joint>
     </xacro:macro>
-    <xacro:macro name="x_link_cylinder" params="name origin_xyz origin_rpy radius length">
+    <xacro:macro name="x_link_cylinder" params="name origin_xyz origin_rpy radius length mass ixx ixy ixz iyy iyz izz">
         <link name="${name}">
+            <inertial>
+                <mass value="${mass}"/>
+                <origin xyz="${origin_xyz}" rpy="${origin_rpy}"/>
+                <inertia ixx="${ixx}" ixy="${ixy}" ixz="${ixz}" iyy="${iyy}" iyz="${iyz}" izz="${izz}"/>
+            </inertial>
+            <collision>
+                <origin xyz="${origin_xyz}" rpy="${origin_rpy}"/>
+                <geometry>
+                    <cylinder radius="${radius}" length="${length}"/>
+                </geometry>
+            </collision>
             <visual>
                 <origin xyz="${origin_xyz}" rpy="${origin_rpy}"/>
@@ -20,6 +31,17 @@
         </link>
     </xacro:macro>
-    <xacro:macro name="x_link_box" params="name origin_xyz origin_rpy size">
+    <xacro:macro name="x_link_box" params="name origin_xyz origin_rpy size mass ixx ixy ixz iyy iyz izz">
         <link name="${name}">
+            <inertial>
+                <mass value="${mass}"/>
+                <origin xyz="${origin_xyz}" rpy="${origin_rpy}"/>
+                <inertia ixx="${ixx}" ixy="${ixy}" ixz="${ixz}" iyy="${iyy}" iyz="${iyz}" izz="${izz}"/>
+            </inertial>
+            <collision>
+               <origin xyz="${origin_xyz}" rpy="${origin_rpy}"/>
+                <geometry>
+                    <box size="${size}"/>
+                </geometry>
+            </collision>
             <visual>
                 <origin xyz="${origin_xyz}" rpy="${origin_rpy}"/>
@@ -30,6 +52,17 @@
         </link>
     </xacro:macro>
-    <xacro:macro name="x_link_ball" params="name origin_xyz origin_rpy radius">
+    <xacro:macro name="x_link_ball" params="name origin_xyz origin_rpy radius mass ixx ixy ixz iyy iyz izz">
         <link name="${name}">
+            <inertial>
+                <mass value="${mass}"/>
+                    <origin xyz="${origin_xyz}" rpy="${origin_rpy}"/>
+                <inertia ixx="${ixx}" ixy="${ixy}" ixz="${ixz}" iyy="${iyy}" iyz="${iyz}" izz="${izz}"/>
+            </inertial>
+            <collision>
+                <origin xyz="${origin_xyz}" rpy="${origin_rpy}"/>
+                <geometry>
+                    <sphere radius="${radius}"/>
+                </geometry>
+            </collision>
             <visual>
                 <origin xyz="${origin_xyz}" rpy="${origin_rpy}"/>

Commit message: Added complete launchfile for Gazebo Added materials for URDF & SDF

File: robot_arm/urdf/jl.xacro (robot description, xacro)
@@ -10,5 +10,5 @@
         </joint>
     </xacro:macro>
-    <xacro:macro name="x_link_cylinder" params="name origin_xyz origin_rpy radius length mass ixx ixy ixz iyy iyz izz">
+    <xacro:macro name="x_link_cylinder" params="name origin_xyz origin_rpy radius length mass ixx ixy ixz iyy iyz izz material">
         <link name="${name}">
             <inertial>
@@ -28,8 +28,9 @@
                     <cylinder radius="${radius}" length="${length}"/>
                 </geometry>
+                <material name="${material}"/>
             </visual>
         </link>
     </xacro:macro>
-    <xacro:macro name="x_link_box" params="name origin_xyz origin_rpy size mass ixx ixy ixz iyy iyz izz">
+    <xacro:macro name="x_link_box" params="name origin_xyz origin_rpy size mass ixx ixy ixz iyy iyz izz material">
         <link name="${name}">
             <inertial>
@@ -49,8 +50,9 @@
                     <box size="${size}"/>
                 </geometry>
+                <material name="${material}"/>
             </visual>
         </link>
     </xacro:macro>
-    <xacro:macro name="x_link_ball" params="name origin_xyz origin_rpy radius mass ixx ixy ixz iyy iyz izz">
+    <xacro:macro name="x_link_ball" params="name origin_xyz origin_rpy radius mass ixx ixy ixz iyy iyz izz material">
         <link name="${name}">
             <inertial>
@@ -70,4 +72,5 @@
                     <sphere radius="${radius}"/>
                 </geometry>
+                <material name="${material}"/>
             </visual>
         </link>

File: robot_arm/urdf/rm.xacro (robot description, xacro)
@@ -3,13 +3,15 @@
     <xacro:include filename="$(find robot_arm)/urdf/jl.xacro"/>
     <xacro:include filename="$(find robot_arm)/urdf/lp.xacro"/>
-    <!-- Opis robota -->
+    <xacro:include filename="$(find robot_arm)/urdf/materials.xacro"/>
+    <!-- Baza -->
     <xacro:x_link_box name="${l00}"
     origin_xyz="0 0 0"  origin_rpy="0 0 0"
-    mass = "2400"
+    mass = "2400" size="2 2 6"
     ixx="8000" ixy="0" ixz="0" iyy="1600" izz="8000" iyz="0"
-    size="2 2 6"/>
+    material="Rust"
+    />
     <!-- Barka, przód tył -->
     <xacro:x_joint name="Shoulder_01" type="revolute"
-    axis="0 1 0"    limit_low="0.87"   limit_up="-2.97" limit_eff="10000"  limit_vel="0.5"
+    axis="0 1 0"    limit_low="0.87"   limit_up="-2.97" limit_eff="1000"  limit_vel="0.5"
     origin_xyz="0 0 2"    origin_rpy="0 0 0"
     parent="${l00}"  child="${l01}"/>
@@ -26,7 +28,7 @@
     <xacro:x_link_box name="${l01}"
     origin_xyz="0 1.5 0"  origin_rpy="0 0 0"
-    mass = "192"
+    mass = "192" size="1 1 1"
     ixx="32" ixy="0" ixz="0" iyy="32" izz="32" iyz="0"
-    size="1 1 1"/>
+    material="Rust" />
     <!-- Bark, od siebie do siebie -->
     <xacro:x_joint name="Shoulder_02" type="revolute"
@@ -46,7 +48,7 @@
     <xacro:x_link_ball name="${l02}"
     origin_xyz="0 0 0" origin_rpy="0 0 0"
-    mass = "40"
+    mass = "40" radius="0.4"
     ixx="0.2" ixy="0" ixz="0" iyy="0.2" izz="0.2" iyz="0"
-    radius="0.4"/>
+    material="Rust" />
     <!-- Ramię, martwy joint -->
     <xacro:x_joint name="Arm_01" type="revolute"
@@ -66,7 +68,7 @@
     <xacro:x_link_cylinder name="${l03}"
     origin_xyz="0 0 0" origin_rpy="0 0 0"
-    mass = "48"
+    mass = "48" radius="0.3" length="1"
     ixx="5.08" ixy="0" ixz="0" iyy="5.08" izz="2.16" iyz="0"
-    radius="0.3" length="1"/>
+    material="Rust" />
     <!-- Łokieć, rotacja -->
     <xacro:x_joint name="Arm_02" type="revolute"
@@ -86,7 +88,7 @@
     <xacro:x_link_ball name="${l04}"
     origin_xyz="0 0 0" origin_rpy="0 0 0"
-    mass = "15"
+    mass = "15" radius="0.3"
     ixx="0.54" ixy="0" ixz="0" iyy="0.54" izz="0.54" iyz="0"
-    radius="0.3"/>
+    material="Rust" />
     <!-- Łokieć, zgięcie-->
     <xacro:x_joint name="Arm_03" type="revolute"
@@ -106,7 +108,7 @@
     <xacro:x_link_cylinder name="${l05}"
     origin_xyz="0 0 -0.4" origin_rpy="0 0 0"
-    mass = "48"
+    mass = "48" radius="0.25" length="0.75"
     ixx="3" ixy="0" ixz="0" iyy="3" izz="2.25" iyz="0"
-    radius="0.25" length="0.75"/>
+    material="Rust" />
     <!-- Nadgarstek, góra dół -->
     <xacro:x_joint name="Wrist" type="revolute"
@@ -126,7 +128,7 @@
     <xacro:x_link_ball name="${l06}"
     origin_xyz="0 0 0" origin_rpy="0 0 0"
-    mass = "15"
+    mass = "15" radius="0.20"
     ixx="0.24" ixy="0" ixz="0" iyy="0.24" izz="0.24" iyz="0"
-    radius="0.20"/>
+    material="Rust" />
     <!-- Nadgarstek, rotacyjny -->
     <xacro:x_joint name="Hand" type="revolute"
@@ -146,7 +148,7 @@
     <xacro:x_link_box name="${l07}"
     origin_xyz="0 0 -0.1"  origin_rpy="0 0 0"
-    mass = "24"
+    mass = "24" size="0.3 0.2 0.4"
     ixx="0.5" ixy="0" ixz="0" iyy="0.26" izz="1.36" iyz="0"
-    size="0.3 0.2 0.4"/>
+    material="Rust" />
      <!-- Palec wskazujący A -->
     <xacro:x_joint name="Finger_01_A" type="revolute"
@@ -166,7 +168,7 @@
     <xacro:x_link_box name="${l08}"
     origin_xyz="0 0 -0.1" origin_rpy="0 0 0"
-    mass = "4"
-    ixx="0.17" ixy="0" ixz="0" iyy="0.00417" izz="0.0542" iyz="0"
-    size="0.1 0.05 0.2"/>
+    mass = "4" size="0.1 0.05 0.2"
+    ixx="0.17" ixy="0" ixz="0" iyy="0.00417" izz="0.0542" iyz="0"
+    material="Rust" />
 <!-- Palec wskazujący B -->
     <xacro:x_joint name="Finger_01_B" type="revolute"
@@ -186,7 +188,7 @@
     <xacro:x_link_box name="${l11}"
     origin_xyz="0 0 -0.1" origin_rpy="0 0 0"
-    mass = "4"
+    mass = "4" size="0.1 0.05 0.2"
     ixx="0.15" ixy="0" ixz="0" iyy="0.0375" izz="0.1275" iyz="0"
-    size="0.1 0.05 0.2"/>
+    material="Rust" />
    <!--  Palec serdeczny A -->
     <xacro:x_joint name="Finger_02_A" type="revolute"
@@ -206,7 +208,7 @@
     <xacro:x_link_box name="${l09}"
     origin_xyz="-0.17 0 -0.1" origin_rpy="0 0 0"
-    mass = "4"
-    ixx="0.17" ixy="0" ixz="0" iyy="0.00417" izz="0.0542" iyz="0"
-    size="0.1 0.05 0.2"/>
+    mass = "4"  size="0.1 0.05 0.2"
+    ixx="0.17" ixy="0" ixz="0" iyy="0.00417" izz="0.0542" iyz="0"
+    material="Rust" />
      <!-- Palec serdeczny B -->
     <xacro:x_joint name="Finger_02_B" type="revolute"
@@ -226,7 +228,7 @@
     <xacro:x_link_box name="${l12}"
     origin_xyz="0 0 -0.1" origin_rpy="0 0 0"
-    mass = "4"
-    ixx="0.17" ixy="0" ixz="0" iyy="0.00417" izz="0.0542" iyz="0"
-    size="0.1 0.05 0.2"/>
+    mass = "4" size="0.1 0.05 0.2"
+    ixx="0.17" ixy="0" ixz="0" iyy="0.00417" izz="0.0542" iyz="0"
+    material="Rust" />
     <!--  Palec kciuk A -->
     <xacro:x_joint name="Finger_03_A" type="revolute"
@@ -246,7 +248,7 @@
     <xacro:x_link_box name="${l10}"
     origin_xyz="-0.05 0 -0.1" origin_rpy="0 0 0"
-    mass = "4"
-    ixx="0.17" ixy="0" ixz="0" iyy="0.00417" izz="0.0542" iyz="0"
-    size="0.1 0.05 0.2"/>
+    mass = "4"  size="0.1 0.05 0.2"
+    ixx="0.17" ixy="0" ixz="0" iyy="0.00417" izz="0.0542" iyz="0"
+    material="Rust" />
      <!-- Palec kciuk B -->
     <xacro:x_joint name="Finger_03_B" type="revolute"
@@ -266,7 +268,7 @@
     <xacro:x_link_box name="${l13}"
     origin_xyz="-0.05 0 -0.1" origin_rpy="0 0 0"
-    mass = "4"
-    ixx="0.17" ixy="0" ixz="0" iyy="0.00417" izz="0.0542" iyz="0"
-    size="0.1 0.05 0.2"/>
+    mass = "4" size="0.1 0.05 0.2"
+    ixx="0.17" ixy="0" ixz="0" iyy="0.00417" izz="0.0542" iyz="0"
+    material="Rust" />
     <gazebo>
         <plugin name="gazebo_ros_control" filename="libgazebo_ros_control.so">

Commit message: fixed everything

File: robot_arm/urdf/jl.xacro (robot description, xacro)
@@ -14,5 +14,5 @@
     <!-- Cylinder -->
 <!--================================================================================-->
-    <xacro:macro name="x_link_cylinder" params="name origin_xyz origin_rpy radius length mass ixx ixy ixz iyy iyz izz material">
+    <xacro:macro name="x_link_cylinder" params="name origin_xyz origin_rpy radius coll_rad length mass ixx ixy ixz iyy iyz izz material">
         <link name="${name}">
             <inertial>
@@ -24,5 +24,5 @@
                 <origin xyz="${origin_xyz}" rpy="${origin_rpy}"/>
                 <geometry>
-                    <cylinder radius="${radius}" length="${length}"/>
+                    <cylinder radius="${coll_rad}" length="${length}"/>
                 </geometry>
             </collision>
@@ -62,5 +62,5 @@
     <!-- Sfera -->
 <!--================================================================================-->
-    <xacro:macro name="x_link_ball" params="name origin_xyz origin_rpy radius mass ixx ixy ixz iyy iyz izz material">
+    <xacro:macro name="x_link_ball" params="name origin_xyz origin_rpy radius coll_rad mass ixx ixy ixz iyy iyz izz material">
         <link name="${name}">
             <inertial>
@@ -72,5 +72,5 @@
                 <origin xyz="${origin_xyz}" rpy="${origin_rpy}"/>
                 <geometry>
-                    <sphere radius="0.1"/>
+                    <sphere radius="${coll_rad}"/>
                 </geometry>
             </collision>

File: robot_arm/urdf/rm.xacro (robot description, xacro)
@@ -15,5 +15,5 @@
 <!--================================================================================-->
     <xacro:x_joint name="Shoulder_01" type="revolute"
-    axis="0 1 0"    limit_low="-2.97"   limit_up="0.87" limit_eff="30000"  limit_vel="1"
+    axis="0 1 0"    limit_low="-2.97"   limit_up="0.87" limit_eff="20000"  limit_vel="0.5"
     origin_xyz="0 0 3"    origin_rpy="0 0 0"
     parent="${l00}"  child="${l01}"/>
@@ -30,11 +30,11 @@
     <xacro:x_link_box name="${l01}"
     origin_xyz="0 1.5 0"  origin_rpy="0 0 0"
-    mass = "192" size="1 0.98 1"
-    ixx="16" iyy="16" izz="16" iyz="0" ixy="0" ixz="0"
+    mass = "250" size="1 1 1"
+    ixx="42" iyy="42" izz="42" iyz="0" ixy="0" ixz="0"
     material="Rust" />
     <!-- Barka, od siebie do siebie -->
 <!--================================================================================-->
     <xacro:x_joint name="Shoulder_02" type="revolute"
-    axis="1 0 0"    limit_low="-0.35"   limit_up="1.6" limit_eff="30000"    limit_vel="1"
+    axis="1 0 0"    limit_low="-0.35"   limit_up="1.6" limit_eff="20000"    limit_vel="0.5"
     origin_xyz="0 2 -0.5"    origin_rpy="0 0 0"
     parent="${l01}"  child="${l02}"/>
@@ -51,6 +51,6 @@
     <xacro:x_link_ball name="${l02}"
     origin_xyz="0 0 0" origin_rpy="0 0 0"
-    mass = "40" radius="0.4"
-    ixx="1.28" iyy="1.28" izz="1.28" iyz="0"  ixy="0" ixz="0"
+    mass = "150" radius="0.4" coll_rad="0.13"
+    ixx="9.6" iyy="9.6" izz="9.6" iyz="0"  ixy="0" ixz="0"
     material="Rust" />
     <!-- Ramię, martwy joint -->
@@ -72,6 +72,6 @@
     <xacro:x_link_cylinder name="${l03}"
     origin_xyz="0 0 0" origin_rpy="0 0 0"
-    mass = "48" radius="0.25" length="1"
-    ixx="17.7" iyy="17.7" izz="1.08" iyz="0"  ixy="0" ixz="0"
+    mass = "120" radius="0.25" coll_rad="0.06" length="1"
+    ixx="10" iyy="10" izz="3.125" iyz="0"  ixy="0" ixz="0"
     material="Rust" />
     <!-- Łokieć, rotacja -->
@@ -93,11 +93,11 @@
     <xacro:x_link_ball name="${l04}"
     origin_xyz="0 0 0" origin_rpy="0 0 0"
-    mass = "15" radius="0.3"
-    ixx="0.54" iyy="0.54" izz="0.54" iyz="0" ixy="0" ixz="0"
+    mass = "40" radius="0.3" coll_rad="0.1"
+    ixx="1.44" iyy="1.44" izz="1.44" iyz="0" ixy="0" ixz="0"
     material="Rust" />
     <!-- Łokieć, zgięcie-->
 <!--================================================================================-->
     <xacro:x_joint name="Arm_03" type="revolute"
-    axis="0 1 0"    limit_low="-2.62"   limit_up="0" limit_eff="20000"    limit_vel="1"
+    axis="0 1 0"    limit_low="-2.62"   limit_up="0" limit_eff="20000"    limit_vel="0.5"
     origin_xyz="0 0 0"    origin_rpy="0 0 0"
     parent="${l04}"  child="${l05}"/>
@@ -114,6 +114,6 @@
     <xacro:x_link_cylinder name="${l05}"
     origin_xyz="0 0 -0.6" origin_rpy="0 0 0"
-    mass = "48" radius="0.2" length="0.75"
-    ixx="10" iyy="10" izz="1.5" iyz="0" ixy="0" ixz="0"
+    mass = "20" radius="0.17" coll_rad="0.04" length="0.75"
+    ixx="3" iyy="3" izz="0.5" iyz="0" ixy="0" ixz="0"
     material="Rust" />
     <!-- Nadgarstek, góra dół -->
@@ -135,6 +135,6 @@
     <xacro:x_link_ball name="${l06}"
     origin_xyz="0 0 -0.05" origin_rpy="0 0 0"
-    mass = "15" radius="0.20"
-    ixx="0.24" iyy="0.24" izz="0.24" iyz="0" ixy="0" ixz="0"
+    mass = "4" radius="0.20" coll_rad="0.06"
+    ixx="0.064" iyy="0.064" izz="0.064" iyz="0" ixy="0" ixz="0"
     material="Rust" />
     <!-- Nadgarstek, rotacyjny -->
@@ -156,6 +156,6 @@
     <xacro:x_link_box name="${l07}"
     origin_xyz="0 0 -0.25"  origin_rpy="0 0 0"
-    mass = "24" size="0.3 0.2 0.4"
-    ixx="0.5" iyy="0.26" izz="4.24" iyz="0"  ixy="0" ixz="0"
+    mass = "10" size="0.3 0.2 0.4"
+    ixx="0.21" iyy="0.11" izz="0.18" iyz="0"  ixy="0" ixz="0"
     material="Rust" />
      <!-- Palec wskazujący A -->
@@ -163,5 +163,5 @@
     <xacro:x_joint name="Finger_01_A" type="revolute"
     axis="1 0 0"    limit_low="-1.57"   limit_up="0.52" limit_eff="10000"    limit_vel="0.5"
-    origin_xyz="0.08 0.08 -0.3"    origin_rpy="0 0 0"
+    origin_xyz="0.08 0.08 -0.5"    origin_rpy="0 0 0"
     parent="${l07}"  child="${l08}"/>
     <transmission name="trans_Finger_01_A">
@@ -178,5 +178,5 @@
     origin_xyz="0 0 -0.1" origin_rpy="0 0 0"
     mass = "4" size="0.1 0.05 0.2"
-    ixx="1.344" iyy="0.014" izz="0.02" iyz="0" ixy="0" ixz="0"
+    ixx="0" iyy="0" izz="0" iyz="0" ixy="0" ixz="0"
     material="Rust" />
     <!-- Palec wskazujący B -->
@@ -184,5 +184,5 @@
     <xacro:x_joint name="Finger_01_B" type="revolute"
     axis="1 0 0"    limit_low="-2.27"   limit_up="0" limit_eff="10000"    limit_vel="0.5"
-    origin_xyz="0 0 -0.2"    origin_rpy="0 0 0"
+    origin_xyz="0 0 -0.25"    origin_rpy="0 0 0"
     parent="${l08}"  child="${l11}"/>
     <transmission name="trans_Finger_01_B">
@@ -199,5 +199,5 @@
     origin_xyz="0 0 -0.1" origin_rpy="0 0 0"
     mass = "4" size="0.1 0.05 0.2"
-    ixx="1.344" iyy="0.014" izz="0.02" iyz="0" ixy="0" ixz="0"
+    ixx="0" iyy="0" izz="0" iyz="0" ixy="0" ixz="0"
     material="Rust" />
    <!--  Palec serdeczny A -->
@@ -205,5 +205,5 @@
     <xacro:x_joint name="Finger_02_A" type="revolute"
     axis="1 0 0"    limit_low="-1.57"   limit_up="0.52" limit_eff="10000"    limit_vel="0.5"
-    origin_xyz="0.08 0.08 -0.3"    origin_rpy="0 0 0"
+    origin_xyz="0.08 0.08 -0.5"    origin_rpy="0 0 0"
     parent="${l07}"  child="${l09}"/>
     <transmission name="trans_Finger_02_A">
@@ -220,5 +220,5 @@
     origin_xyz="-0.17 0 -0.1" origin_rpy="0 0 0"
     mass = "4"  size="0.1 0.05 0.2"
-    ixx="1.344" iyy="0.014" izz="0.02" iyz="0" ixy="0" ixz="0"
+    ixx="0" iyy="0" izz="0" iyz="0" ixy="0" ixz="0"
     material="Rust" />
      <!-- Palec serdeczny B -->
@@ -226,5 +226,5 @@
     <xacro:x_joint name="Finger_02_B" type="revolute"
     axis="1 0 0"    limit_low="-2.27"   limit_up="0" limit_eff="10000"    limit_vel="0.5"
-    origin_xyz="-0.17 0 -0.2"    origin_rpy="0 0 0"
+    origin_xyz="-0.17 0 -0.25"    origin_rpy="0 0 0"
     parent="${l09}"  child="${l12}"/>
     <transmission name="trans_Finger_02_B">
@@ -241,5 +241,5 @@
     origin_xyz="0 0 -0.1" origin_rpy="0 0 0"
     mass = "4" size="0.1 0.05 0.2"
-    ixx="1.344" iyy="0.014" izz="0.02" iyz="0" ixy="0" ixz="0"
+    ixx="0" iyy="0" izz="0" iyz="0" ixy="0" ixz="0"
     material="Rust" />
     <!--  Palec kciuk A -->
@@ -247,5 +247,5 @@
     <xacro:x_joint name="Finger_03_A" type="revolute"
     axis="1 0 0"    limit_low="-0.7"   limit_up="1.57" limit_eff="10000"    limit_vel="0.5"
-    origin_xyz="0.08 -0.06 -0.3"    origin_rpy="0 0 0"
+    origin_xyz="0.08 -0.06 -0.5"    origin_rpy="0 0 0"
     parent="${l07}"  child="${l10}"/>
     <transmission name="trans_Finger_03_A">
@@ -262,5 +262,5 @@
     origin_xyz="-0.05 0 -0.1" origin_rpy="0 0 0"
     mass = "4"  size="0.1 0.05 0.2"
-    ixx="1.344" iyy="0.014" izz="0.02" iyz="0" ixy="0" ixz="0"
+    ixx="0" iyy="0" izz="0" iyz="0" ixy="0" ixz="0"
     material="Rust" />
      <!-- Palec kciuk B -->
@@ -268,5 +268,5 @@
     <xacro:x_joint name="Finger_03_B" type="revolute"
     axis="1 0 0"    limit_low="0"   limit_up="1.6" limit_eff="10000"    limit_vel="0.5"
-    origin_xyz="0 0 -0.2"    origin_rpy="0 0 0"
+    origin_xyz="0 0 -0.25"    origin_rpy="0 0 0"
     parent="${l10}"  child="${l13}"/>
     <transmission name="trans_Finger_03_B">
@@ -283,5 +283,5 @@
     origin_xyz="-0.05 0 -0.1" origin_rpy="0 0 0"
     mass = "4" size="0.1 0.05 0.2"
-    ixx="1.344" iyy="0.014" izz="0.02" iyz="0" ixy="0" ixz="0"
+    ixx="0" iyy="0" izz="0" iyz="0" ixy="0" ixz="0"
     material="Rust" />
     <!-- Plugin -->
